File: hardware/ProjectAlienArbReplacement.kicad_sch (KiCad schematic)
At the start: 9 parts, among them J1 Bumper Connector, J3 Left Motor Connector, J4 Right Motor Connector, J5 Pixels Connector, J6 Ultrasonic Connector, J7 Micro USB, U1 4021

Commit message: Added I2C multiplexer
Parts:
- added J8: I2C Multiplexer, Adafruit_5664_Shield:Adafruit_5664_Shield, symbol Connector:Conn_01x05_Socket
- J7: footprint Connector_PinHeader_2.54mm:PinHeader_1x05_P2.54mm_Vertical -> Adafruit_1833_Shield:Adafruit_1833_Shield
Changed lines of the file:
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@@
 			)
 		)
-		(property "Footprint" "Connector_PinHeader_2.54mm:PinHeader_1x05_P2.54mm_Vertical"
+		(property "Footprint" "Adafruit_1833_Shield:Adafruit_1833_Shield"
 			(at 46.99 171.45 0)
 			(effects
@@
 					(unit 1)
 				)
+			)
+		)
+	)
+	(symbol
+		(lib_id "Connector:Conn_01x05_Socket")
+		(at 146.05 176.53 0)
+		(unit 1)
+		(exclude_from_sim no)
+		(in_bom yes)
+		(on_board yes)
+		(dnp no)
+		(fields_autoplaced yes)
+		(property "Reference" "J8"
+			(at 147.32 175.2599 0)
+			(effects
+				(font
+					(size 1.27 1.27)
+				)
+				(justify left)
+			)
+		)
+		(property "Value" "I2C Multiplexer"
+			(at 147.32 177.7999 0)
+			(effects
+				(font
+					(size 1.27 1.27)
+				)
+				(justify left)
+			)
+		)
+		(property "Footprint" "Adafruit_5664_Shield:Adafruit_5664_Shield"
+			(at 146.05 176.53 0)
+			(effects
+				(font
+					(size 1.27 1.27)
+				)
+				(hide yes)
+			)
+		)
+		(property "Datasheet" "~"
+			(at 146.05 176.53 0)
+			(effects
+				(font
+					(size 1.27 1.27)
+				)
+				(hide yes)
+			)
+		)
+		(property "Description" "Generic connector, single row, 01x05, script generated"
+			(at 146.05 176.53 0)
+			(effects
+				(font
+					(size 1.27 1.27)
+				)
+				(hide yes)
+			)
+		)
+		(pin "4"
+		)
+		(pin "3"
+		)
+		(pin "1"
+		)
+		(pin "5"
+		)
+		(pin "2"
+		)
+		(instances
+			(project "ProjectAlienArbReplacement"
+				(path "/170b00d5-17da-40d3-a37d-b29c3db0afc1"
+					(reference "J8")
+					(unit 1)
+				)

Commit message: Added motor driver
Parts:
- added M1: ~, DFRobot_DC_Motor_Driver_Shield:DFRobot_DC_Motor_Driver_Shield, symbol DFRobot_DC_Motor_Driver_Shield:DFRobot_DC_Motor_Driver_Shield
Connections:
- net GND: now also M1.5 (GND), M1.8 (GND)
- net at A1.12 (D9): now also M1.2 (PMW1)
- net at A1.13 (D10): now also M1.3 (PMW2)
- net at A1.19 (A0): now also M1.1 (DIR1)
- net at A1.20 (A1): now also M1.4 (DIR2)
Other:
- moved on the sheet: J7
