File: hardware/ProjectAlienMainBoard.kicad_pcb (KiCad board)
At the start: 2 copper layers, 69.1 x 100.6 mm, 53 parts, among them J1 Bumper, J10 Excess GPIO Pins, J3 Left Motor, J4 Right Motor, J5 Pixels, J6 Ultrasonic, J7 Micro USB, J8 I2C Multiplexer, J9 Voltage Breakout, Q1 2N3904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

Commit message: Added title to PCB
Other:
- board text added: "(Autonomous Labyrinth Investigator, Explorer, Navigator)"
- board text added: "A.L.I.E.N."
- board text added: "By Harry Boyd"
- board text added: "Project"
- board text added: "github.com/HBoyd255/project-alien"
