File: hardware/ProjectALIENMainBoard.kicad_pcb (KiCad board)
At the start: 2 copper layers, 69.1 x 100.6 mm, 53 parts, among them J1 Bumper, J10 Excess GPIO Pins, J3 Left Motor, J4 Right Motor, J5 Pixels, J6 Ultrasonic, J7 Micro USB, J8 I2C Multiplexer, J9 Voltage Breakout, Q1 2N3904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

Commit message: Tidied up traces
Connections:
- U1 pad 11: BUMPER_DATA -> unconnected-(U1-DS-Pad11)
- U1 pad 3: unconnected-(U1-Q7-Pad3) -> BUMPER_DATA
Routing:
- net ENC2A: track 46.8 -> 43.5 mm, vias 2 -> 0
- net Net-(A1-~{RESET}-Pad3): track 34.6 -> 31.7 mm
- net USONIC_TRIG: track 68.3 -> 70.0 mm
- net PWM1: track 30.3 -> 28.6 mm
- net PWM2: track 29.0 -> 30.4 mm
- net GND: vias 24 -> 28

Commit message: Fixed direction of connectors
Routing:
- net Net-(J1-Pin_7): track 13.9 -> 1.94 mm
- net Net-(J1-Pin_8): track 13.9 -> 1.94 mm
- net Net-(J1-Pin_6): track 13.9 -> 1.94 mm
- net Net-(J1-Pin_4): track 6.28 -> 0.00 mm
- net Net-(J1-Pin_3): track 6.28 -> 0.00 mm
- net Net-(J1-Pin_2): track 6.28 -> 0.00 mm
- net Net-(J1-Pin_9): track 6.28 -> 1.94 mm
- net Net-(J1-Pin_5): track 6.28 -> 1.94 mm
- net GND: vias 28 -> 24

Commit message: Fixed connector Issues
Parts:
- J3, J4, J6: moved to F.Cu
- moved U1 20.8 mm to (150.6, 101.5), turned to 0 degrees
- moved R12 19.3 mm to (153.0, 101.6), turned to 0 degrees
- moved R11 14.3 mm to (155.8, 104.0), turned to 180 degrees
- moved J4 14.2 mm to (162.0, 77.2)
- moved J3 12.7 mm to (114.8, 90.2)
- moved R5 11.8 mm to (153.0, 116.8), turned to 0 degrees
- moved R10 9.22 mm to (155.8, 106.6), turned to 180 degrees
- moved J6 7.65 mm to (114.8, 66.1)
- moved R6 7.02 mm to (153.0, 114.2), turned to 0 degrees
- moved R8 5.00 mm to (153.0, 109.2), turned to 0 degrees
- moved R9 4.38 mm to (155.8, 109.2), turned to 180 degrees
- moved R7 3.47 mm to (153.0, 111.8), turned to 0 degrees
- moved TP19 1.57 mm to (158.6, 84.8)
- moved TP20 1.51 mm to (158.6, 87.4)
Routing:
- net +3.3V: track 251.1 -> 214.2 mm
- net GND: track 17.1 -> 0.00 mm, vias 24 -> 33
- net Net-(J1-Pin_2): track 0.00 -> 15.7 mm
- net Net-(J1-Pin_3): track 0.00 -> 15.3 mm
- net Net-(J1-Pin_4): track 0.00 -> 15.3 mm
- net Net-(J1-Pin_5): track 1.94 -> 15.4 mm
- net Net-(J1-Pin_9): track 1.94 -> 14.7 mm
- net SHIFT_REG_LOAD: track 57.7 -> 48.8 mm
- net Net-(J1-Pin_6): track 1.94 -> 6.22 mm
- net Net-(J1-Pin_8): track 1.94 -> 6.22 mm
- net Net-(J1-Pin_7): track 1.94 -> 6.20 mm
- net ENC2A: track 43.5 -> 47.6 mm
- net M2-: track 21.5 -> 24.3 mm
- net SHIFT_REG_CLOCK: track 60.2 -> 57.8 mm, vias 1 -> 0
- net M2+: track 21.5 -> 23.4 mm
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Other:
- board text added: "Project A.L.I.E.N. Main Board V1.1 24/08/2024 Harry Boyd"
- board text removed: "Project A.L.I.E.N. Main Board V1.0 15/08/2024 Harry Boyd"

Commit message: Updated designators
Parts:
- renumbered A1 to U1, M1 to U2, U1 to U3
